File: hardware/NES_V5/NEScartridge.kicad_sch (KiCad schematic)
At the start: 39 parts, among them J1 Conn_02x36_Top_Bottom, U1 TXS0108EPW, U10 TXS0108EPW, U11 TXS0108EPW, U2 TXS0108EPW, U5 TXS0108EPW, U6 TXS0108EPW, U7 TXS0108EPW, U8 TXS0108EPW, U9 TXS0108EPW

Commit message: Corrected DRC errors/warning on V5
Connections:
- no-connect marks 3 -> 20
Changed lines of the file:
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@@
   (junction (at 250.19 76.2) (diameter 0) (color 0 0 0 0)
   )
+  (no_connect (at 72.39 163.83))
   (no_connect (at 121.92 344.17))
+  (no_connect (at 53.34 373.38))
   (no_connect (at 53.34 340.36))
+  (no_connect (at 53.34 370.84))
+  (no_connect (at 72.39 148.59))
+  (no_connect (at 52.07 146.05))
+  (no_connect (at 228.6 111.76))
+  (no_connect (at 52.07 161.29))
+  (no_connect (at 248.92 111.76))
+  (no_connect (at 248.92 106.68))
+  (no_connect (at 228.6 109.22))
+  (no_connect (at 52.07 148.59))
+  (no_connect (at 52.07 163.83))
+  (no_connect (at 228.6 106.68))
+  (no_connect (at 248.92 109.22))
+  (no_connect (at 66.04 383.54))
   (no_connect (at 53.34 342.9))
+  (no_connect (at 72.39 161.29))
+  (no_connect (at 72.39 146.05))
   (wire (pts (xy 241.3 130.81) (xy 250.19 130.81))
     (stroke (width 0) (type default))
